File: CY8C4248AZI-L475/CY8C4248AZI-L475.kicad_pcb (KiCad board)
At the start: 2 copper layers, 37.7 x 33.2 mm, 26 parts, among them J1 USB_C_Receptacle_USB2.0_16P, J3 Conn_02x10_Odd_Even, J4 Conn_02x09_Odd_Even, J7 Conn_02x10_Odd_Even, U1 *

Commit message: Teardrop
Routing:
- net GNDA: track 14.5 -> 16.1 mm

Commit message: Update
Parts:
- J1: moved to B.Cu
- moved R2 4.35 mm to (160.0, 60.8), turned to 0 degrees
- moved R1 3.42 mm to (160.0, 59.4), turned to 0 degrees
- moved R3 2.83 mm to (159.1, 56.4)
- moved R4 2.83 mm to (159.1, 57.9)
- turned J1 to -90 degrees
Connections:
- net Net-(J1-D+-PadA6) renamed D+
- net Net-(J1-D--PadA7) renamed D-
Routing:
- net /VBUS: track 27.2 -> 19.6 mm, vias 0 -> 2
- net Net-(J1-CC1): track 2.30 -> 5.77 mm, vias 0 -> 1
- net Net-(U1-D+_P13_0): track 5.96 -> 3.49 mm
- net Net-(U1-D-_P13_1): track 6.10 -> 3.76 mm
- net D-: track 5.85 -> 7.34 mm, vias 2 -> 1
- net Net-(J1-CC2): track 2.09 -> 2.67 mm, vias 0 -> 1
- net D+: track 6.64 -> 6.93 mm, vias 0 -> 1
- net GNDD: vias 13 -> 11
