File: CY8C4248AZI-L475/CY8C4248AZI-L475.kicad_sch (KiCad schematic)
At the start: 19 parts, among them J1 USB_C_Receptacle_USB2.0_16P, U1 *

Commit message: Add
Parts:
- added J3, J7: Conn_02x10_Odd_Even, Connector_PinSocket_2.54mm:PinSocket_2x10_P2.54mm_Vertical, symbol Connector_Generic:Conn_02x10_Odd_Even
- added J4: Conn_02x09_Odd_Even, Connector_PinSocket_2.54mm:PinSocket_2x09_P2.54mm_Vertical, symbol Connector_Generic:Conn_02x09_Odd_Even
- C1, C10, C11, C2, C3, C4, C5, C6, C7, C8, C9: footprint (none) -> Capacitor_SMD:C_0603_1608Metric
- J1: footprint (none) -> Connector_USB:USB_C_Receptacle_HRO_TYPE-C-31-M-12
- NT1, NT2: footprint (none) -> NetTie:NetTie-3_SMD_Pad0.5mm
- R1, R2, R3, R4: footprint (none) -> Resistor_SMD:R_0603_1608Metric
- U1: footprint (none) -> CY8C4248AZI-L475:TQFP50P1200X1200X160-64N
Connections:
- net +5V: now also J7.1 (Pin_1)
- net GND: now also J7.2 (Pin_2); no longer J1.A1 (GND), J1.A12 (GND), J1.B1 (GND), J1.B12 (GND), J1.S1 (SHIELD), R1.1, R2.1
- net GNDD: now also J1.A1 (GND), J1.A12 (GND), J1.B1 (GND), J1.B12 (GND), J1.S1 (SHIELD), R1.1, R2.1
- net P0_0: now also J3.3 (Pin_3)
- net P0_1: now also J3.6 (Pin_6)
- net P0_2: now also J3.5 (Pin_5)
- net P0_3: now also J3.8 (Pin_8)
- net P0_4: now also J3.7 (Pin_7)
- net P0_5: now also J3.10 (Pin_10)
- net P0_6: now also J3.9 (Pin_9)
- net P0_7: now also J3.12 (Pin_12)
- net P1_0: now also J3.17 (Pin_17)
- net P1_1: now also J3.19 (Pin_19)
- net P1_2: now also J4.2 (Pin_2)
- net P1_3: now also J4.1 (Pin_1)
- net P1_4: now also J4.4 (Pin_4)
- net P1_5: now also J4.3 (Pin_3)
- net P1_6: now also J4.6 (Pin_6)
- net P1_7_VREF: now also J4.5 (Pin_5)
- net P2_0: now also J4.8 (Pin_8)
- net P2_1: now also J4.7 (Pin_7)
- net P2_2: now also J4.10 (Pin_10)
- net P2_3: now also J4.9 (Pin_9)
- net P2_4: now also J4.12 (Pin_12)
- net P2_5: now also J4.11 (Pin_11)
- net P2_6: now also J4.14 (Pin_14)
- net P2_7: now also J4.13 (Pin_13)
- net P3_0: now also J7.18 (Pin_18)
- net P3_1: now also J7.17 (Pin_17)
- net P3_2_SWDIO: now also J7.16 (Pin_16)
- net P3_3_SWDCLK: now also J7.15 (Pin_15)
- net P3_4: now also J7.14 (Pin_14)
- net P3_5: now also J7.13 (Pin_13)
- net P3_6: now also J7.12 (Pin_12)
- net P3_7: now also J7.11 (Pin_11)
- net P4_0: now also J7.10 (Pin_10)
- net P4_1: now also J7.9 (Pin_9)
- net P4_2: now also J7.8 (Pin_8)
- net P4_3: now also J7.7 (Pin_7)
- net P4_4: now also J7.6 (Pin_6)
- net P4_5: now also J7.5 (Pin_5)
- net P4_6: now also J7.4 (Pin_4)
- net P5_0: now also J3.14 (Pin_14)
- net P5_1: now also J3.13 (Pin_13)
- net P5_2: now also J3.16 (Pin_16)
- net P5_3: now also J3.15 (Pin_15)
- net P5_5: now also J3.18 (Pin_18)
- net P6_0: now also J4.16 (Pin_16)
- net P6_1: now also J4.15 (Pin_15)
- net P6_2: now also J4.18 (Pin_18)
- net P6_4_P12_0: now also J4.17 (Pin_17)
- net P6_5_P12_1: now also J7.20 (Pin_20)
- net P7_0: now also J3.1 (Pin_1)
- net P7_1: now also J3.4 (Pin_4)
- net VBUS: now also J7.3 (Pin_3)
- net VBUS_P13_2: now also J3.2 (Pin_2)
- net ~{XRES}: now also J3.11 (Pin_11)
- no-connect marks 2 -> 4

Commit message: Update
Connections:
- net D+: now reaches J1.A6 (D+), J1.B6 (D+), R4.2
- net D-: now reaches J1.A7 (D-), J1.B7 (D-), R3.2
Changed lines of the file:
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@@
+		)
+	)
+	(global_label "D-"
+		(shape input)
+		(at 133.35 85.09 180)
+		(fields_autoplaced yes)
+		(effects
+			(font
+				(size 1.27 1.27)
+			)
+			(justify right)
+		)
+		(property "Intersheetrefs" "${INTERSHEET_REFS}"
+			(at 127.5224 85.09 0)
+			(effects
+				(font
+					(size 1.27 1.27)
+				)
+				(justify right)
+				(hide yes)
+			)
+		)
+	)
+	(global_label "D+"
+		(shape input)
+		(at 133.35 90.17 180)
+		(fields_autoplaced yes)
+		(effects
+			(font
+				(size 1.27 1.27)
+			)
+			(justify right)
+		)
+		(property "Intersheetrefs" "${INTERSHEET_REFS}"
+			(at 127.5224 90.17 0)
+			(effects
+				(font
+					(size 1.27 1.27)
+				)
+				(justify right)
+				(hide yes)
+			)
 		)
 	)
