File: ATmega32U4/ATmega32U4.kicad_pcb (KiCad board)
At the start: 2 copper layers, 38.3 x 30.6 mm, 26 parts, among them J1 USB_C_Receptacle_USB2.0_16P, J2 Conn_01x15, J3 Conn_01x15, U1 ATmega32U4-A, Y1 16M

Commit message: Update
Parts:
- D1, D2: footprint Diode_SMD:D_0603_1608Metric -> Library:CDBVRL140-HF
- moved D2 0.76 mm to (121.7, 45.6)
- moved D1 0.67 mm to (121.7, 46.9)
