File: ATmega32U4/ATmega32U4.kicad_sch (KiCad schematic)
At the start: 26 parts, among them J1 USB_C_Receptacle_USB2.0_16P, J2 Conn_01x15, J3 Conn_01x15, U1 ATmega32U4-A, Y1 16M

Commit message: Update
Parts:
- C10, C11, C12: LCSC (none) -> C386081
- D1, D2: footprint Diode_SMD:D_0603_1608Metric -> Library:CDBVRL140-HF; LCSC (none) -> C3758192
- J1: LCSC (none) -> C165948
- Y1: LCSC (none) -> C19078192
Changed lines of the file:
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@@
+			)
+		)
+		(property "LCSC" "C386081"
+			(at 92.71 27.94 0)
+			(effects
+				(font
+					(size 1.27 1.27)
+				)
+				(hide yes)
 			)
 		)
@@
 			)
 		)
+		(property "LCSC" "C386081"
+			(at 154.94 30.48 0)
+			(effects
+				(font
+					(size 1.27 1.27)
+				)
+				(hide yes)
+			)
+		)
 		(pin "1"
 		)
@@
 		)
 		(property "Description" "USB 2.0-only 16P Type-C Receptacle connector"
+			(at 27.94 38.1 0)
+			(effects
+				(font
+					(size 1.27 1.27)
+				)
+				(hide yes)
+			)
+		)
+		(property "LCSC" "C165948"
 			(at 27.94 38.1 0)
 			(effects
@@
 			)
 		)
+		(property "LCSC" "C19078192"
+			(at 43.18 90.17 0)
+			(effects
+				(font
+					(size 1.27 1.27)
+				)
+				(hide yes)
+			)
+		)
 		(pin "2"
 		)
@@
 		)
 		(property "Description" "Unpolarized capacitor, small symbol"
+			(at 146.05 30.48 0)
+			(effects
+				(font
+					(size 1.27 1.27)
+				)
+				(hide yes)
+			)
+		)
+		(property "LCSC" "C386081"
 			(at 146.05 30.48 0)
 			(effects
@@
 			)
 		)
-		(property "Footprint" "Diode_SMD:D_0603_1608Metric"
+		(property "Footprint" "Library:CDBVRL140-HF"
 			(at 81.28 29.21 0)
 			(effects
@@
 			)
 		)
+		(property "LCSC" "C3758192"
+			(at 81.28 29.21 0)
+			(effects
+				(font
+					(size 1.27 1.27)
+				)
+				(hide yes)
+			)
+		)
 		(pin "1"
 		)
@@
 			)
 		)
-		(property "Footprint" "Diode_SMD:D_0603_1608Metric"
+		(property "Footprint" "Library:CDBVRL140-HF"
 			(at 81.28 24.13 0)
 			(effects
@@
 			(at 81.28 24.13 0)
 			(effects
+				(font
+					(size 1.27 1.27)
+				)
+				(hide yes)
+			)
+		)
+		(property "LCSC" "C3758192"
+			(at 81.28 24.13 0)
+			(effects
